Commit message: temporary dummy inertia values to pass gz fortress parsing

File: pal_gripper_description/urdf/gripper.urdf.xacro (robot description, xacro)
@@ -54,9 +54,10 @@
   <link name="${name}_right_finger_link">
     <inertial>
-      <origin rpy="0 0 0" xyz="-0.004470 0.010766 -0.121013" />
-      <mass value="0.109980" />
-      <inertia ixx="0.000232" ixy="-0.000005" ixz="-0.000032"
-               iyy="0.000224" iyz="0.000036"
-               izz="0.000029" />
+      <!-- <origin rpy="0 0 0" xyz="-0.004470 0.010766 -0.121013" /> -->
+      <!-- <mass value="0.109980" /> -->
+      <!-- <inertia ixx="0.000232" ixy="-0.000005" ixz="-0.000032" iyy="0.000224" iyz="0.000036" izz="0.000029" /> -->
+     <origin xyz="0.0 0.0 0.0" rpy="0.0 0.0 0.0"/>
+     <mass value="1.0"/>
+     <inertia ixx="0.01" ixy="0.0" ixz="0.0" iyy="0.01" iyz="0.0" izz="0.01"/>
     </inertial>
     <visual>
@@ -92,9 +93,10 @@
   <link name="${name}_left_finger_link">
     <inertial>
-      <origin rpy="0 0 0" xyz="-0.004470 0.010766 -0.121013" />
-      <mass value="0.109980" />
-      <inertia ixx="0.000232" ixy="-0.000005" ixz="-0.000032"
-               iyy="0.000224" iyz="0.000036"
-               izz="0.000029" />
+      <origin xyz="0.0 0.0 0.0" rpy="0.0 0.0 0.0"/>
+      <mass value="1.0"/>
+      <inertia ixx="0.01" ixy="0.0" ixz="0.0" iyy="0.01" iyz="0.0" izz="0.01"/>
+      <!-- <origin rpy="0 0 0" xyz="-0.004470 0.010766 -0.121013" /> -->
+      <!-- <mass value="0.109980" /> -->
+      <!-- <inertia ixx="0.000232" ixy="-0.000005" ixz="-0.000032" iyy="0.000224" iyz="0.000036" izz="0.000029" /> -->
     </inertial>
     <visual>
